File: LP_MSPM0C1104-EB-V1.1/LP_MSPM0C1104-EB-V1.1.kicad_pcb (KiCad board)
At the start: 2 copper layers, 58.4 x 40.6 mm, 65 parts, among them J1 PWR, J1 SSQ-110-03-F-S, J2 KLINE, J2 SSQ-110-03-F-S, J3 SSQ-102-03-F-S, J4 PEC03SAAN, J5 PEC03SAAN, Q1 PDTC123JT, Q2 PBSS4041NT,215, Q4 PDTC123JT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

Commit message: update value
Parts:
- R26, R8: value 220R -> 560R
Connections:
- net KLINE renamed LIN
- net V_BAT renamed VIN

Commit message: export gerber file
Parts:
- added R13: 0R, Resistor_SMD:R_0603_1608Metric, F.Cu at (151.1, 97.1)
- added R15: 0R, Resistor_SMD:R_0603_1608Metric, F.Cu at (158.7, 97.1)
- added R16: 0R, Resistor_SMD:R_0603_1608Metric, F.Cu at (162.2, 102.3)
- added R17: 0R, Resistor_SMD:R_0603_1608Metric, F.Cu at (162.9, 110.1)
- added R18: 0R, Resistor_SMD:R_0603_1608Metric, F.Cu at (147.0, 123.8)
- added R19: 0R, Resistor_SMD:R_0603_1608Metric, F.Cu at (143.1, 108.7)
- added R20: 0R, Resistor_SMD:R_0603_1608Metric, F.Cu at (139.3, 111.8)
- C2, C20, C5, C6, C7, C8: value 0.1uF/50V -> 0.1uF
- C9: value 2.2uF/25V -> 2.2uF
- J2: value KLINE -> LIN
- R11: value 47R-1/2W -> 47R
- U4: value AP7380-33W5-7 -> AP7380
- moved R21 15.2 mm to (151.1, 93.1)
- moved Q5 11.4 mm to (154.3, 91.9)
- moved Q6 11.4 mm to (154.3, 95.9)
- moved C5 2.44 mm to (146.6, 89.6), turned to -90 degrees
- moved D5 2.41 mm to (157.9, 92.7), turned to -90 degrees
- moved Q4 1.10 mm to (162.0, 95.9)
- moved R14 1.05 mm to (161.8, 89.2)
- moved Q2 1.05 mm to (162.0, 91.9)
- moved BZ1 0.35 mm to (131.3, 105.4)
- renumbered SW3 to SW1, SW1 to SW2, SW2 to SW3
Connections:
- net 12V renamed Net-(D6-K)
- C2 pad 1: PA18_A7_BP -> /KEY1
- C7 pad 1: PA16 -> /KEY0
- C8 pad 1: PA22_A4 -> /KEY2
- Q1 pad 1: PA6 -> Net-(Q1-B)
- Q4 pad 1: PA27_UART_TX_A0 -> Net-(Q4-B)
- Q6 pad 3: PA26_UART_RX_A1 -> Net-(Q6-C)
- Q8 pad 3: PA11_BP -> Net-(Q8-C)
- R10 pad 2: PA22_A4 -> /KEY2
- R4 pad 2: PA16 -> /KEY0
- R6 pad 2: PA18_A7_BP -> /KEY1
- SW1 pad 2: PA22_A4 -> /KEY2
- SW2 pad 2: PA18_A7_BP -> /KEY1
- SW3 pad 2: PA16 -> /KEY0
Routing:
- net PA26_UART_RX_A1: track 43.0 -> 27.1 mm
- net PA22_A4: track 56.0 -> 41.3 mm
- net /KEY2: track 0.00 -> 13.7 mm
- net PA18_A7_BP: track 29.3 -> 15.9 mm
- net LIN: track 29.0 -> 16.5 mm
- net /KEY0: track 0.00 -> 12.0 mm
- net /KEY1: track 0.00 -> 11.8 mm
- net PA16: track 26.6 -> 18.3 mm, vias 0 -> 1
- net PA11_BP: track 19.3 -> 14.4 mm
- net PA27_UART_TX_A0: track 39.3 -> 35.1 mm
- net Net-(Q8-C): track 0.00 -> 3.41 mm
- net Net-(Q2-B): track 10.3 -> 7.13 mm, vias 2 -> 0
- net Net-(Q1-B): track 0.00 -> 2.60 mm
- net Net-(Q6-C): track 0.00 -> 2.55 mm
- net Net-(Q4-B): track 0.00 -> 1.61 mm
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