File: LP_MSPM0C1104-EB-V1.1/LP_MSPM0C1104-EB-V1.1.kicad_sch (KiCad schematic)
At the start: 60 parts, among them J1 PWR, J2 KLINE, Q1 PDTC123JT, Q2 PBSS4041NT,215, Q4 PDTC123JT, Q5 PDTC123JT, Q6 PDTC123JT, Q8 PDTC123JT, SW1 SW_Push, SW2 SW_Push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

Commit message: update value
Parts:
- BZ1: IKY-MPN IKY-LC004 -> (none); Manufacturer P/N BRT1209PF-06 -> (none)
- C1, C14, C3, C4: IKY-MPN IKY-MA002 -> (none); Manufacturer P/N CL05B104KB5NNNC -> (none)
- C15: IKY-MPN IKY-B032 -> (none); Manufacturer P/N CL10A475KP8NNNC -> (none)
- C17: IKY-MPN IKY-B008 -> (none); Manufacturer P/N 08051C822KAT2A -> (none)
- C18: IKY-MPN IKY-B016 -> (none); Manufacturer P/N CL10C102JB8NNNC -> (none)
- C2, C20, C5, C6, C7, C8: value 0.1uF/50V -> 0.1uF; IKY-MPN IKY-MA002 -> (none); Manufacturer P/N CL05B104KB5NNNC -> (none)
- C9: value 2.2uF/25V -> 2.2uF; IKY-MPN IKY-PTM007 -> (none); Manufacturer P/N GRM188R61E225KA12D -> (none)
- D1: IKY-MPN IKY-MA040 -> (none); Manufacturer P/N BZX384-C3V6,115 -> (none)
- D10, D3: IKY-MPN IKY-B009 -> (none); Manufacturer P/N 1N4148W-7-F -> (none)
- D11: IKY-MPN IKY-LC019 -> (none); Manufacturer P/N SMAZ30-13-F -> (none)
- D4: IKY-MPN IKY-B001 -> (none); Manufacturer P/N S1M-13-F -> (none)
- D5, D6: IKY-MPN IKY-CF002 -> (none); Manufacturer P/N SMAJ20CA-13-F -> (none)
- Q1, Q4, Q6, Q8: IKY-MPN IKY-B015 -> (none); Manufacturer P/N PDTC123JT,215 -> (none)
- Q2: IKY-MPN IKY-MA021 -> (none); Manufacturer P/N PBSS4041NT,215 -> (none)
- Q5: IKY-MPN IKY-B013 -> (none); Manufacturer P/N PMBT2222A,215 -> (none)
- R1, R2: IKY-MPN IKY-MA039 -> (none); Manufacturer P/N RC0402JR-074K7L -> (none)
- R10, R4, R5, R6: IKY-MPN IKY-GPS023 -> (none); Manufacturer P/N RC0402FR-0710KL -> (none)
- R11: value 47R-1/2W -> 47R; IKY-MPN IKY-PTM016 -> (none); Manufacturer P/N RC1210JR-0747RL -> (none)
- R12: IKY-MPN IKY-LC013 -> (none); Manufacturer P/N RC1206JR-071KL -> (none)
- R14, R21: IKY-MPN IKY-B018 -> (none); Manufacturer P/N RC0603JR-0722KL -> (none)
- R22: IKY-MPN IKY-B023 -> (none); Manufacturer P/N RC0603FR-07220KL -> (none)
- R24, R9: IKY-MPN IKY-PTK003 -> (none); Manufacturer P/N RC0402JR-07220RL -> (none)
- R25: IKY-MPN IKY-TR020 -> (none); Manufacturer P/N RC0402FR-07470KL -> (none)
- R26, R8: value 220R -> 560R; IKY-MPN IKY-PTK003 -> (none); Manufacturer P/N RC0402JR-07220RL -> (none)
- R27, R28: IKY-MPN IKY-RD034 -> (none); Manufacturer P/N RC0402JR-07100KL -> (none)
- R3: IKY-MPN IKY-TR022 -> (none); Manufacturer P/N RC0402FR-07100KL -> (none)
- R7: IKY-MPN IKY-LC032 -> (none); Manufacturer P/N RC0805JR-07100RL -> (none)
- U4: value AP7380-33W5-7 -> AP7380; IKY-MPN IKY-SK029 -> (none); Manufacturer P/N AP7380-33W5-7 -> (none)
- U6: IKY-MPN IKY-B003 -> (none); Manufacturer P/N LM358ADT -> (none)
Connections:
- net KLINE renamed LIN
- net V_BAT renamed VIN
Other:
- moved on the sheet: C15, C17, C18, D10, D11, L1, Q5, Q6, R21, R22, R24, R25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

Commit message: export gerber file
Parts:
- added R13, R15, R16, R17, R18, R19, R20: 0R, Resistor_SMD:R_0603_1608Metric, symbol Device:R_Small_US
- J2: value KLINE -> LIN
- renumbered SW3 to SW1, SW1 to SW2, SW2 to SW3
Connections:
- net PA11_BP: now also R20.1; no longer Q8.3 (C)
- net PA16: now also R16.1; no longer C7.1, R4.2, SW3.2
- net PA18_A7_BP: now also R17.1; no longer C2.1, R6.2, SW2.2
- net PA22_A4: now also R18.1; no longer C8.1, R10.2, SW1.2
- net PA26_UART_RX_A1: now also R13.1; no longer Q6.3 (C)
- net PA27_UART_TX_A0: now also R15.1; no longer Q4.1 (B)
- net PA6: now also R19.2; no longer Q1.1 (B)
- net 12V: no longer names the net of C6.1, C9.1, D6.1 (K), R11.1, U4.1 (VIN), U4.3 (EN)
- new net: Q8.3 (C), R20.2
- new net: Q4.1 (B), R15.2
- new net: Q6.3 (C), R13.2
- new net: Q1.1 (B), R19.1
- new net KEY0: C7.1, R16.2, R4.2, SW3.2
- new net KEY1: C2.1, R17.2, R6.2, SW2.2
- new net KEY2: C8.1, R10.2, R18.2, SW1.2
Other:
- note added: "16V Max"
- moved on the sheet: R11, TP1
